File: PCB/pcb/pcb/pcb.kicad_pcb (KiCad board)
At the start: 2 copper layers, 65 x 56 mm, 5 parts, among them P1 Conn_02x20_Odd_Even

Commit message: V0.7 finish the schematic that close #4
Parts:
- removed MK1, MK2, MK3, MK4: M2.5, MountingHole:MountingHole_2.7mm_M2.5
- removed P1: Conn_02x20_Odd_Even, Connector_PinSocket_2.54mm:PinSocket_2x20_P2.54mm_Vertical
Other:
- board outline removed
- board text removed: "CAMERA"
- board text removed: "DISPLAY"
- board text removed: "RASPBERRY-PI 40-PIN ADDON BOARD VIEW FROM TOP NOTE: P1 SHOULD BE FITTED ON THE REVERSE OF THE BOARD ADD EDGE CUTS FROM CAMERA AND DISPLAY PORTS AS REQUIRED"
- board text removed: "RJ45"
- board text removed: "USB"
