File: PCB/pcb/pcb/_autosave-pcb.kicad_pcb (KiCad board)
At the start: 2 copper layers, 70.9 x 62.7 mm, 28 parts

Commit message: V0.8 pcb Finished this closes #9 and closes #8
Parts:
- removed MK2: M2.5, MountingHole:MountingHole_2.7mm_M2.5
- moved MK1 65.1 mm to (244.2, 114.7)
- moved MK3 59.1 mm to (180.6, 169.9)
- moved MK4 47.8 mm to (180.9, 114.0)
- moved limit_swtich2 24.2 mm to (242.9, 168.5)
- moved limit_swtich3 23.6 mm to (232.0, 168.5)
- moved Motor_power_plug1 22.4 mm to (191.2, 142.1)
- moved limit_swtich1 16.1 mm to (242.9, 161.4)
- moved Motor2 13.8 mm to (192.5, 160.5)
- moved motor2_plug1 13.5 mm to (182.1, 164.3)
- moved limit_swtich4 11.7 mm to (231.8, 161.4)
- moved R2 8.76 mm to (211.2, 161.4), turned to 270 degrees
- moved R1 6.35 mm to (216.3, 161.4), turned to 270 degrees
- moved Arduino_power_plug1 3.84 mm to (234.0, 123.8)
- moved R3 3.75 mm to (206.1, 161.4), turned to 270 degrees
- moved R4 2.65 mm to (221.3, 161.4), turned to 270 degrees
Connections:
- Arduino_Nano1 pad 13: Limit_switch1 -> Net-(Arduino_Nano1-Pad13)
- Arduino_Nano1 pad 19: Net-(Arduino_Nano1-Pad19) -> Limit_switch1
- Arduino_Nano1 pad 4: GND -> Net-(Arduino_Nano1-Pad4)
- Arduino_power_plug1 pad 2: Net-(Arduino_power_plug1-Pad2) -> GND
- Motor_power_plug1 pad 2: Net-(Motor_power_plug1-Pad2) -> GND_motor
Routing:
- net GND: track 44.1 -> 0.00 mm
- net +5V: track 271.8 -> 233.0 mm
- net GND_motor: track 71.1 -> 41.4 mm
- net Limit_switch4: track 33.2 -> 14.0 mm
- net EN_motor2: track 14.0 -> 27.9 mm
- net Limit_switch3: track 19.8 -> 33.7 mm
- net Limit_switch2: track 30.4 -> 44.2 mm
- net Step_motor2: track 8.05 -> 15.2 mm
- net Dir_motor2: track 8.05 -> 14.5 mm
- net Vmot_1: track 45.5 -> 42.4 mm
- net Limit_switch1: track 45.1 -> 42.3 mm
- net Step_motor1: track 20.7 -> 21.8 mm
- net Dir_motor1: track 21.3 -> 22.2 mm
- net S_LED1: track 11.9 -> 12.8 mm
- net S_LED2: track 8.33 -> 8.97 mm
Other:
- net class Default: clearance 0.2 -> 0.25; trace_width 0.2 -> 0.4
- net class Power: clearance 0.2 -> 0.25; trace_width 0.5 -> 0.4
- rule trace_clearance: 0.2 -> 0.25
- rule trace_min: 0.1524 -> 0.2
