File: PCB/pcb/pcb/_autosave-pcb.sch (KiCad schematic (older format))
At the start: 27 parts

Commit message: V0.8 pcb Finished this closes #9 and closes #8
Connections:
- net +5V: no longer Arduino_Nano1.27 (+5V)
- no-connect marks 5 -> 7
Changed lines of the file:
@@
 	3100 1500 3100 1600
 Connection ~ 3100 1600
-$Comp
-L power:+5V #PWR?
-U 1 1 5F6E3F0F
-P 6450 3300
-F 0 "#PWR?" H 6450 3150 50  0001 C CNN
-F 1 "+5V" H 6465 3473 50  0000 C CNN
-F 2 "" H 6450 3300 50  0001 C CNN
-F 3 "" H 6450 3300 50  0001 C CNN
-	1    6450 3300
-	1    0    0    -1
-$EndComp
-Wire Wire Line
-	6450 3300 6450 3400
+NoConn ~ 6450 3400
+NoConn ~ 6350 3400
 $EndSCHEMATC
